File: flight_controller/core.sch (EAGLE design)
At the start: 100 parts, among them J1 M02, J10 MOLEX-2POS, J11 MOLEX-2POS, J12 MOLEX-2POS, J13 MOLEX-3POS, J14 MOLEX-3POS, J15 MOLEX-4POS, J16 MOLEX-3POS, J17 M03, J18 M04, J19 MOLEX-3POS, J2 MOLEX-2POS, J20 MOLEX-4POS, J21 MOLEX-2POS, J22 MOLEX-2POS, J3 MOLEX-2POS, J4 MOLEX-2POS, J5 MOLEX-2POS, J6 MOLEX-2POS, J7 MOLEX-2POS, J8 MOLEX-2POS, Q1 EM6K1, Q10 EM6K1, Q11 EM6K1, Q2 EM6K1, Q3 MOSFET-PCHANNEL-AON6407, Q7 EM6K1, Q8 EM6K1, U2 MEAS-MS5611, U3 USD-SOCKETNEW, U4 STM32F405, U5 MIC5219 3.3V, U6 MPU-9250-QFN-24-NP, Y1 16MHz

Commit message: Renumber schematic.
Parts:
- removed J22: MOLEX-2POS, aerial:MOLEX-2POS
- removed LED14, LED15: OSRAM-MULTILED-RGB, OSURC_LED:OSRAM-MULTILED-RGB
- removed Q8: EM6K1, OSURC_DiscreteSemi:MOSFET-NCHANNEL-DUAL-EM6K1
- removed R35, R36, R38, R43, R48: 1K, SparkFun:RESISTOR0603-RES
- removed R37: 20K, SparkFun-Passives:RESISTOR0603-RES
- removed U6: MPU-9250-QFN-24-NP, OSURC_Sensors:MPU-9250-QFN-24-NP
- added J9: MOLEX-3POS, aerial:MOLEX-3POS
- added LED2, LED4: YELLOW, SparkFun-LED:LED0603
- added Q6: EM6K1, OSURC_DiscreteSemi:MOSFET-NCHANNEL-DUAL-EM6K1
- added R11, R13: 100, SparkFun-Passives:RESISTOR0603-RES
- added R12, R23: 680, SparkFun-Passives:RESISTOR0603-RES
- added R14: 120, SparkFun-Passives:RESISTOR0603-RES
- added R15: 165, SparkFun-Passives:RESISTOR0603-RES
- added U1: STM32F405, OSURC_DigitalIC:STM32F405
- C1: value 0.1uF -> 18pF; device SparkFun-Capacitors:0.1UF-25V-5%(0603) -> SparkFun-Capacitors:18PF-50V-5%(0603)
- C10, C13: value 2.2uF -> 0.1uF; device SparkFun-Capacitors:2.2UF-10V-20%(0603) -> SparkFun-Capacitors:0.1UF-25V-5%(0603)
- C11: value 0.1uF -> 2.2uF; device SparkFun-Capacitors:0.1UF-25V-5%(0603) -> SparkFun-Capacitors:2.2UF-10V-20%(0603)
- C12: value 10nF -> 2.2uF; device SparkFun-Capacitors:10NF/10000PF-50V-10%(0603) -> SparkFun-Capacitors:2.2UF-10V-20%(0603)
- C15: value 18pF -> 0.1uF; device SparkFun-Capacitors:18PF-50V-5%(0603) -> SparkFun-Capacitors:0.1UF-25V-5%(0603)
- C16: value 18pF -> 10nF; device SparkFun-Capacitors:18PF-50V-5%(0603) -> SparkFun-Capacitors:10NF/10000PF-50V-10%(0603)
- C2: value 1nF -> 18pF; device SparkFun-Capacitors:1NF/1000PF-50V-10%(0603) -> SparkFun-Capacitors:18PF-50V-5%(0603)
- C5: value 0.1uF -> 1nF; device SparkFun-Capacitors:0.1UF-25V-5%(0603) -> SparkFun-Capacitors:1NF/1000PF-50V-10%(0603)
- J13, J14: value MOLEX-3POS -> MOLEX-2POS; device aerial:MOLEX-3POS -> aerial:MOLEX-2POS
- J15: value MOLEX-4POS -> MOLEX-2POS; device aerial:MOLEX-4POS -> aerial:MOLEX-2POS
- J18: value M04 -> MOLEX-4POS; device OSURC_Connectors:M04 -> aerial:MOLEX-4POS
- J19: value MOLEX-3POS -> M04; device aerial:MOLEX-3POS -> OSURC_Connectors:M04
- J20: value MOLEX-4POS -> MOLEX-3POS; device aerial:MOLEX-4POS -> aerial:MOLEX-3POS
- J21: value MOLEX-2POS -> MOLEX-4POS; device aerial:MOLEX-2POS -> aerial:MOLEX-4POS
- J4: value MOLEX-2POS -> MOLEX-3POS; device aerial:MOLEX-2POS -> aerial:MOLEX-3POS
- LED10, LED11: value YELLOW -> ORANGE
- LED5: value ORANGE -> OSRAM-MULTILED-RGB; device SparkFun-LED:LED0603 -> OSURC_LED:OSRAM-MULTILED-RGB
- LED6: value ORANGE -> GREEN
- LED7: value ORANGE -> RED
- LED8: value GREEN -> OSRAM-MULTILED-RGB; device SparkFun-LED:LED0603 -> OSURC_LED:OSRAM-MULTILED-RGB
- LED9: value RED -> ORANGE
- Q3: value MOSFET-PCHANNEL-AON6407 -> EM6K1; device OSURC_DiscreteSemi:MOSFET-PCHANNEL-AON6407 -> OSURC_DiscreteSemi:MOSFET-NCHANNEL-DUAL-EM6K1
- Q7: value EM6K1 -> MOSFET-PCHANNEL-AON6407; device OSURC_DiscreteSemi:MOSFET-NCHANNEL-DUAL-EM6K1 -> OSURC_DiscreteSemi:MOSFET-PCHANNEL-AON6407
- R1, R17: value 20K -> 680
- R10: value 120 -> 680
- R16, R18: value 20K -> 100
- R2: value 1K -> 680
- R24: value 100 -> 680
- R25: value 100 -> 20K; device SparkFun-Passives:RESISTOR0603-RES -> SparkFun:RESISTOR0603-RES
- R26: value 120 -> 20K
- R27, R29, R30: value 680 -> 20K
- R28: value 165 -> 20K
- R3, R4, R7: value 680 -> 1K; device SparkFun-Passives:RESISTOR0603-RES -> SparkFun:RESISTOR0603-RES
- R31: value 680 -> 1K5
- R32: value 1K1 -> 20K
- R33: value 100 -> 1K5
- R34: value 100 -> 1K
- R5: value 20K -> 1K; device SparkFun-Passives:RESISTOR0603-RES -> SparkFun:RESISTOR0603-RES
- R6: value 1K5 -> 1K; device SparkFun-Passives:RESISTOR0603-RES -> SparkFun:RESISTOR0603-RES
- R8: value 20K -> 120; device SparkFun:RESISTOR0603-RES -> SparkFun-Passives:RESISTOR0603-RES
- R9: value 1K5 -> 1K1
- U3: value USD-SOCKETNEW -> MPU-9250-QFN-24-NP; device SparkFun-Connectors:USD-SOCKETNEW -> OSURC_Sensors:MPU-9250-QFN-24-NP
- U4: value STM32F405 -> MIC5219 3.3V; device OSURC_DigitalIC:STM32F405 -> SparkFun-PowerIC:V_REG_MIC52193.3V
- U5: value MIC5219 3.3V -> USD-SOCKETNEW; device SparkFun-PowerIC:V_REG_MIC52193.3V -> SparkFun-Connectors:USD-SOCKETNEW
- renumbered LED12 to LED1, LED13 to LED3, Q10 to Q4, Q11 to Q5, R44 to R19, R45 to R20, R46 to R21, R47 to R22
Connections:
- net 3.3V: now also C10.1, C13.1, C15.1, C16.1, C4.+, R1.1, R25.2, R3.2, R31.2, R33.2, R34.2, U1.POWER.VBAT, U1.POWER.VDD@19, U1.POWER.VDD@32, U1.POWER.VDD@48, U1.POWER.VDD@64, U1.POWER.VDDA, U3.RESV@1, U3.VDD, U3.VDDIO, U4.OUT, U5.VCC; no longer C1.1, C11.1, C12.1, C3.+, C5.1, R2.2, R31.1, R48.2, R6.2, R8.2, R9.2, U3.VCC, U4.POWER.VBAT, U4.POWER.VDD@19, U4.POWER.VDD@32, U4.POWER.VDD@48, U4.POWER.VDD@64, U4.POWER.VDDA, U5.OUT, U6.RESV@1, U6.VDD, U6.VDDIO
- net 5V: now also C3.+, J19.1, J4.2, J9.2, Q7.S, R11.1, R13.1, R14.1, R16.1, R18.1, R8.1, R9.1, U4.EN, U4.IN; no longer C4.+, J13.2, J14.2, J18.1, Q3.S, R10.1, R24.1, R25.1, R26.1, R32.1, R33.1, R34.1, U5.EN, U5.IN
- net ADC1: now also R26.1, R27.1, U1.GPIO.PC0; no longer R1.1, R5.1, U4.GPIO.PC0
- net ADC1-IN: now also J4.1, R26.2; no longer J13.1, R1.2
- net ADC2: now also R28.1, R29.1, U1.GPIO.PC1; no longer R16.1, R17.1, U4.GPIO.PC1
- net ADC2-IN: now also J9.1, R28.2; no longer J14.1, R16.2
- net F4-VCAP-1: now also C11.1, U1.POWER.VCAP_2; no longer C10.1, U4.POWER.VCAP_2
- net F4-VCAP-2: now also C12.1, U1.POWER.VCAP_1; no longer C13.1, U4.POWER.VCAP_1
- net GND: now also J13.2, J14.2, J15.2, J19.4, J20.3, J4.3, J9.3, LED2.C, LED4.C, Q2B.S, Q3A.S, Q3B.S, Q6A.S, Q7.G, R27.2, R29.2, R30.2, R32.2, U1.POWER.VSS@18, U1.POWER.VSS@63, U1.POWER.VSSA, U3.FSYNC, U3.RESV@20, U4.GND, U5.SHIELD@1, U5.SHIELD@3; no longer J13.3, J14.3, J15.4, J19.3, J20.2, J22.2, J4.2, LED5.C, LED8.C, Q3.G, Q7A.S, Q7B.S, Q8A.S, Q8B.S, R17.2, R18.2, R37.2, R5.2, U3.SHIELD@1, U3.SHIELD@3, U4.POWER.VSS@18, U4.POWER.VSS@63, U4.POWER.VSSA, U6.FSYNC, U6.GND, U6.RESV@20
- net I2C2-SCL: now also R31.1, U1.GPIO.PB10; no longer R6.1, U4.GPIO.PB10
- net I2C2-SDA: now also R33.1, U1.GPIO.PB11; no longer R9.1, U4.GPIO.PB11
- net KILL: now also Q1A.G, Q1B.G, Q2A.G, Q2B.G, R15.1, R3.1; no longer Q7A.G, Q7B.G, Q8A.G, Q8B.G, R28.1, R48.1
- net MIC-BP: now also C5.1, U4.BP; no longer C2.1, U5.BP
- net MPU9250-REGOUT: now also U3.REGOUT; no longer U6.REGOUT
- net N$12: now also LED5.B+, R13.2; no longer LED14.B+, R25.2
- net N$15: now also LED8.R+, R14.2; no longer LED15.R+, R26.2
- net N$16: now also LED8.G+, R16.2; no longer LED15.G+, R33.2
- net N$19: now also LED8.B+, R18.2; no longer LED15.B+, R34.2
- net N$2: now also LED9.A, R17.2; no longer LED5.A, R3.2
- net N$3: now also LED10.A, R23.2; no longer LED6.A, R4.2
- net N$34: now also LED6.A, R12.2; no longer LED8.A, R27.2
- net N$35: now also LED7.A, R15.2; no longer LED9.A, R28.2
- net N$36: now also LED2.A, R2.2; no longer LED10.A, R29.2
- net N$37: now also LED4.A, R10.2; no longer LED11.A, R30.2
- net N$38: now also R1.2; no longer R31.2
- net N$39: now also R9.2; no longer R32.2
- net N$4: now also LED11.A, R24.2; no longer LED7.A, R7.2
- net N$5: now also LED5.B-, LED8.B-, Q3A.D; no longer LED14.B-, LED15.B-, Q1A.D
- net N$6: now also LED5.G-, LED8.G-, Q3B.D; no longer LED14.G-, LED15.G-, Q1B.D
- net N$7: now also LED5.R-, LED8.R-, Q6A.D; no longer LED14.R-, LED15.R-, Q2A.D
- net N$8: now also LED5.R+, R8.2; no longer LED14.R+, R10.2
- net N$9: now also LED5.G+, R11.2; no longer LED14.G+, R24.2
- net OSC-IN: now also C1.1, U1.GPIO.PH0; no longer C15.1, U4.GPIO.PH0
- net OSC-OUT: now also C2.1, U1.GPIO.PH1; no longer C16.1, U4.GPIO.PH1
- net OTG-HS-DM: now also U1.GPIO.PB14; no longer U4.GPIO.PB14
- net OTG-HS-DP: now also U1.GPIO.PB15; no longer U4.GPIO.PB15
- net OTG-HS-ID: now also U1.GPIO.PB12; no longer U4.GPIO.PB12
- net PA12: now also R17.1, U1.GPIO.PA12; no longer R3.1, U4.GPIO.PA12
- net PA15: now also R23.1, U1.GPIO.PA15; no longer R4.1, U4.GPIO.PA15
- net PA4: now also J3.1, U1.GPIO.PA4; no longer J11.1, U4.GPIO.PA4
- net PA5: now also J8.1, U1.GPIO.PA5; no longer J12.1, U4.GPIO.PA5
- net PB2: now also R24.1, U1.GPIO.PB2; no longer R7.1, U4.GPIO.PB2
- net PC4: now also J12.1, U1.GPIO.PC4; no longer J21.1, U4.GPIO.PC4
- net PC5: now also J15.1, U1.GPIO.PC5; no longer J22.1, U4.GPIO.PC5
- net RST: now also J21.1, R25.1, U1.GPIO.NRST; no longer J20.1, R8.1, U4.GPIO.NRST
- net SDIO-CK: now also U1.GPIO.PC12, U5.SCK; no longer U3.SCK, U4.GPIO.PC12
- net SDIO-CMD: now also U1.GPIO.PD2, U5.DI; no longer U3.DI, U4.GPIO.PD2
- net SDIO-D0: now also U1.GPIO.PC8, U5.DO; no longer U3.DO, U4.GPIO.PC8
- net SDIO-D1: now also U1.GPIO.PC9, U5.RSV; no longer U3.RSV, U4.GPIO.PC9
- net SDIO-D2: now also U1.GPIO.PC10, U5.NC; no longer U3.NC, U4.GPIO.PC10
- net SDIO-D3: now also U1.GPIO.PC11, U5.CS; no longer U3.CS, U4.GPIO.PC11
- net SPI1-MISO: now also R30.1, U1.GPIO.PB4, U3.AD0/SDO; no longer R18.1, U4.GPIO.PB4, U6.AD0/SDO
- net SPI1-MOSI: now also U1.GPIO.PB5, U3.SDA/SDI; no longer U4.GPIO.PB5, U6.SDA/SDI
- net SPI1-SCK: now also U1.GPIO.PB3, U3.SCL/SCLK; no longer U4.GPIO.PB3, U6.SCL/SCLK
- net SPI2-MISO: now also J18.2, R32.1, U1.GPIO.PC2; no longer J15.2, R37.1, U4.GPIO.PC2
- net SPI2-MOSI: now also J18.3, U1.GPIO.PC3; no longer J15.3, U4.GPIO.PC3
- net SPI2-SCK: now also J18.1, U1.GPIO.PB13; no longer J15.1, U4.GPIO.PB13
- net SPISS-MPU9250: now also U1.GPIO.PC14, U3.NCS; no longer U4.GPIO.PC14, U6.NCS
- net SPISS-MS5611: now also U1.GPIO.PC13; no longer U4.GPIO.PC13
- net SPISS-UNUSED: now also U1.GPIO.PC15; no longer U4.GPIO.PC15
- net SWCLK: now also J21.4, U1.GPIO.PA14; no longer J20.4, U4.GPIO.PA14
- net SWDIO: now also J21.3, U1.GPIO.PA13; no longer J20.3, U4.GPIO.PA13
- net TIM1-CH1: now also R4.2, U1.GPIO.PA8; no longer R35.2, U4.GPIO.PA8
- net TIM1-CH1-K: now also Q1A.D, R4.1; no longer Q7A.D, R35.1
- net TIM1-CH2: now also R5.2, U1.GPIO.PA9; no longer R36.2, U4.GPIO.PA9
- net TIM1-CH2-K: now also J6.1, Q1B.D, R5.1; no longer J2.1, Q7B.D, R36.1
- net TIM1-CH3: now also R6.2, U1.GPIO.PA10; no longer R38.2, U4.GPIO.PA10
- net TIM1-CH3-K: now also J10.1, Q2A.D, R6.1; no longer J3.1, Q8A.D, R38.1
- net TIM1-CH4: now also R7.2, U1.GPIO.PA11; no longer R43.2, U4.GPIO.PA11
- net TIM1-CH4-K: now also J13.1, Q2B.D, R7.1; no longer J4.1, Q8B.D, R43.1
- net TIM3-CH1-RSSI: now also R12.1, U1.GPIO.PA6; no longer R27.1, U4.GPIO.PA6
- net TIM3-CH2-STSR: now also Q6A.G, U1.GPIO.PA7; no longer Q2A.G, U4.GPIO.PA7
- net TIM3-CH3-STSG: now also Q3B.G, U1.GPIO.PB0; no longer Q1B.G, U4.GPIO.PB0
- net TIM3-CH4-STSB: now also Q3A.G, U1.GPIO.PB1; no longer Q1A.G, U4.GPIO.PB1
- net TIM4-CH1: now also U1.GPIO.PB6; no longer U4.GPIO.PB6
- net TIM4-CH1-K: now also J2.1; no longer J5.1
- net TIM4-CH2: now also U1.GPIO.PB7; no longer U4.GPIO.PB7
- net TIM4-CH2-K: now also J7.1; no longer J6.1
- net TIM4-CH3: now also U1.GPIO.PB8; no longer U4.GPIO.PB8
- net TIM4-CH3-K: now also J11.1; no longer J7.1
- net TIM4-CH4: now also U1.GPIO.PB9; no longer U4.GPIO.PB9
- net TIM4-CH4-K: now also J14.1; no longer J8.1
- net UART2-RX-XBEE: now also R10.1, U1.GPIO.PA3; no longer R30.1, U4.GPIO.PA3
- net UART2-TX-XBEE: now also R2.1, U1.GPIO.PA2; no longer R29.1, U4.GPIO.PA2
- net UART4-RX: now also J20.2, U1.GPIO.PA1; no longer J19.2, U4.GPIO.PA1
- net UART4-TX: now also J20.1, U1.GPIO.PA0_WKUP; no longer J19.1, U4.GPIO.PA0_WKUP
- net UART6-RX-GPS: now also J19.3, U1.GPIO.PC7; no longer J18.3, U4.GPIO.PC7
- net UART6-TX-GPS: now also J19.2, U1.GPIO.PC6; no longer J18.2, U4.GPIO.PC6
- net USD-CD: now also R34.1, U5.SHIELD@2, U5.SHIELD@4; no longer R2.1, U3.SHIELD@2, U3.SHIELD@4
- net VIN: now also J5.1, Q7.D; no longer J10.1, Q3.D
Other:
- moved on the sheet: C1, C10, C11, C12, C13, C15, C16, C2, C3, C4, C5, C6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
