File: flight_controller/core.brd (EAGLE design)
At the start: 100 parts, among them J1 M02, J10 MOLEX-2POS, J11 MOLEX-2POS, J12 MOLEX-2POS, J13 MOLEX-3POS, J14 MOLEX-3POS, J15 MOLEX-4POS, J16 MOLEX-3POS, J17 M03, J18 M04, J19 MOLEX-3POS, J2 MOLEX-2POS, J20 MOLEX-4POS, J21 MOLEX-2POS, J22 MOLEX-2POS, J3 MOLEX-2POS, J4 MOLEX-2POS, J5 MOLEX-2POS, J6 MOLEX-2POS, J7 MOLEX-2POS, J8 MOLEX-2POS, Q1 EM6K1, Q10 EM6K1, Q11 EM6K1, Q2 EM6K1, Q3 MOSFET-PCHANNEL-AON6407, Q7 EM6K1, Q8 EM6K1, U2 MEAS-MS5611, U3 USD-SOCKETNEW, U4 STM32F405, U5 MIC5219 3.3V, U6 MPU-9250-QFN-24-NP, Y1 16MHz

Commit message: Renumber schematic.
Parts:
- removed J22: MOLEX-2POS, aerial:MOLEX-2MM-MICROLATCH-2POS-RA
- removed LED14, LED15: OSRAM-MULTILED-RGB, OSURC_LED:PLCC-6
- removed Q8: EM6K1, OSURC_DiscreteSemi:SOT-666
- removed R35, R36, R38, R43, R48: 1K, SparkFun:0603-RES
- removed R37: 20K, SparkFun-Passives:0603-RES
- removed U6: MPU-9250-QFN-24-NP, OSURC_Sensors:QFN-24-NP
- added J9: MOLEX-3POS, aerial:MOLEX-2MM-MICROLATCH-3POS-RA
- added LED2, LED4: YELLOW, SparkFun-LED:LED-0603
- added Q6: EM6K1, OSURC_DiscreteSemi:SOT-666
- added R11, R13: 100, SparkFun-Passives:0603-RES
- added R12, R23: 680, SparkFun-Passives:0603-RES
- added R14: 120, SparkFun-Passives:0603-RES
- added R15: 165, SparkFun-Passives:0603-RES
- added U1: STM32F405, OSURC_DigitalIC:LQFP-64-STM32F405
- C1: value 0.1uF -> 18pF
- C10, C13: value 2.2uF -> 0.1uF
- C11: value 0.1uF -> 2.2uF
- C12: value 10nF -> 2.2uF
- C15: value 18pF -> 0.1uF
- C16: value 18pF -> 10nF
- C2: value 1nF -> 18pF
- C5: value 0.1uF -> 1nF
- J13, J14: value MOLEX-3POS -> MOLEX-2POS; device aerial:MOLEX-2MM-MICROLATCH-3POS-RA -> aerial:MOLEX-2MM-MICROLATCH-2POS-RA
- J15: value MOLEX-4POS -> MOLEX-2POS; device aerial:MOLEX-2MM-MICROLATCH-4POS-RA -> aerial:MOLEX-2MM-MICROLATCH-2POS-RA
- J18: value M04 -> MOLEX-4POS; device OSURC_Connectors:MOLEX-2MM-MICROLATCH-4POS-RA -> aerial:MOLEX-2MM-MICROLATCH-4POS-RA
- J19: value MOLEX-3POS -> M04; device aerial:MOLEX-2MM-MICROLATCH-3POS-RA -> OSURC_Connectors:MOLEX-2MM-MICROLATCH-4POS-RA
- J20: value MOLEX-4POS -> MOLEX-3POS; device aerial:MOLEX-2MM-MICROLATCH-4POS-RA -> aerial:MOLEX-2MM-MICROLATCH-3POS-RA
- J21: value MOLEX-2POS -> MOLEX-4POS; device aerial:MOLEX-2MM-MICROLATCH-2POS-RA -> aerial:MOLEX-2MM-MICROLATCH-4POS-RA
- J4: value MOLEX-2POS -> MOLEX-3POS; device aerial:MOLEX-2MM-MICROLATCH-2POS-RA -> aerial:MOLEX-2MM-MICROLATCH-3POS-RA
- LED10, LED11: value YELLOW -> ORANGE
- LED5: value ORANGE -> OSRAM-MULTILED-RGB; device SparkFun-LED:LED-0603 -> OSURC_LED:PLCC-6
- LED6: value ORANGE -> GREEN
- LED7: value ORANGE -> RED
- LED8: value GREEN -> OSRAM-MULTILED-RGB; device SparkFun-LED:LED-0603 -> OSURC_LED:PLCC-6
- LED9: value RED -> ORANGE
- Q3: value MOSFET-PCHANNEL-AON6407 -> EM6K1; device OSURC_DiscreteSemi:DFN5X6 -> OSURC_DiscreteSemi:SOT-666
- Q7: value EM6K1 -> MOSFET-PCHANNEL-AON6407; device OSURC_DiscreteSemi:SOT-666 -> OSURC_DiscreteSemi:DFN5X6
- R1, R17: value 20K -> 680
- R10: value 120 -> 680
- R16, R18: value 20K -> 100
- R2: value 1K -> 680
- R24: value 100 -> 680
- R25: value 100 -> 20K; device SparkFun-Passives:0603-RES -> SparkFun:0603-RES
- R26: value 120 -> 20K
- R27, R29, R30: value 680 -> 20K
- R28: value 165 -> 20K
- R3, R4, R7: value 680 -> 1K; device SparkFun-Passives:0603-RES -> SparkFun:0603-RES
- R31: value 680 -> 1K5
- R32: value 1K1 -> 20K
- R33: value 100 -> 1K5
- R34: value 100 -> 1K
- R5: value 20K -> 1K; device SparkFun-Passives:0603-RES -> SparkFun:0603-RES
- R6: value 1K5 -> 1K; device SparkFun-Passives:0603-RES -> SparkFun:0603-RES
- R8: value 20K -> 120; device SparkFun:0603-RES -> SparkFun-Passives:0603-RES
- R9: value 1K5 -> 1K1
- U3: value USD-SOCKETNEW -> MPU-9250-QFN-24-NP; device SparkFun-Connectors:MICRO-SD-SOCKET-PP -> OSURC_Sensors:QFN-24-NP
- U4: value STM32F405 -> MIC5219 3.3V; device OSURC_DigitalIC:LQFP-64-STM32F405 -> SparkFun-PowerIC:SOT23-5
- U5: value MIC5219 3.3V -> USD-SOCKETNEW; device SparkFun-PowerIC:SOT23-5 -> SparkFun-Connectors:MICRO-SD-SOCKET-PP
- moved U3 685.0 mm to (-249.9, -594.9)
- moved R25 420.0 mm to (-13.3, -182.7)
- moved R8 414.8 mm to (-223.8, -540.1)
- moved LED8 377.4 mm to (-222.5, -537.0)
- moved R10 369.0 mm to (-36.0, -222.5)
- moved LED11 365.7 mm to (-214.8, -522.8)
- moved LED7 362.7 mm to (-30.4, -210.5)
- moved LED10 360.0 mm to (-211.9, -519.7)
- moved LED9 360.0 mm to (-214.8, -519.7)
- moved LED6 357.1 mm to (-33.3, -210.5)
- moved C2 338.3 mm to (-187.5, -506.7)
- moved R29 316.6 mm to (-187.5, -490.4)
- moved R32 316.1 mm to (-187.5, -496.4)
- moved R28 312.5 mm to (-187.5, -487.4)
- moved R30 310.4 mm to (-187.5, -493.4)
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- renumbered LED12 to LED1, LED13 to LED3, Q10 to Q4, Q11 to Q5, R44 to R19, R45 to R20, R46 to R21, R47 to R22
Connections:
- net 3.3V: now also C10.1, C13.1, C15.1, C16.1, C4.A, R1.1, R25.2, R3.2, R31.2, R33.2, R34.2, U1.1, U1.13, U1.19, U1.32, U1.48, U1.64, U3.1, U3.13, U3.8, U4.5, U5.4; no longer C1.1, C11.1, C12.1, C3.A, C5.1, R2.2, R31.1, R48.2, R6.2, R8.2, R9.2, U3.4, U4.1, U4.13, U4.19, U4.32, U4.48, U4.64, U5.5, U6.1, U6.13, U6.8
- net 5V: now also C3.A, J19.1, J4.2, J9.2, Q7.1, Q7.2, Q7.3, R11.1, R13.1, R14.1, R16.1, R18.1, R8.1, R9.1, U4.1, U4.3; no longer C4.A, J13.2, J14.2, J18.1, Q3.1, Q3.2, Q3.3, R10.1, R24.1, R25.1, R26.1, R32.1, R33.1, R34.1, U5.1, U5.3
- net ADC1: now also R26.1, R27.1, U1.8; no longer R1.1, R5.1, U4.8
- net ADC1-IN: now also J4.1, R26.2; no longer J13.1, R1.2
- net ADC2: now also R28.1, R29.1, U1.9; no longer R16.1, R17.1, U4.9
- net ADC2-IN: now also J9.1, R28.2; no longer J14.1, R16.2
- net F4-VCAP-1: now also C11.1, U1.47; no longer C10.1, U4.47
- net F4-VCAP-2: now also C12.1, U1.31; no longer C13.1, U4.31
- net GND: now also J13.2, J14.2, J15.2, J19.4, J20.3, J4.3, J9.3, LED2.C, LED4.C, Q2.4, Q3.1, Q6.1, R27.2, R29.2, R30.2, R32.2, U1.12, U1.18, U1.63, U3.11, U3.18, U3.20, U4.2, U5.6, U5.GND1, U5.GND3; no longer J13.3, J14.3, J15.4, J19.3, J20.2, J22.2, J4.2, LED5.C, LED8.C, Q7.1, Q8.1, Q8.4, R17.2, R18.2, R37.2, R5.2, U3.6, U3.GND1, U3.GND3, U4.12, U4.18, U4.63, U5.2, U6.11, U6.18, U6.20
- net I2C2-SCL: now also R31.1, U1.29; no longer R6.1, U4.29
- net I2C2-SDA: now also R33.1, U1.30; no longer R9.1, U4.30
- net KILL: now also Q1.2, Q1.5, Q2.2, Q2.5, R15.1, R3.1; no longer Q7.2, Q7.5, Q8.2, Q8.5, R28.1, R48.1
- net MIC-BP: now also C5.1, U4.4; no longer C2.1, U5.4
- net MPU9250-REGOUT: now also U3.10; no longer U6.10
- net N$12: now also LED5.A1, R13.2; no longer LED14.A1, R25.2
- net N$15: now also LED8.A2, R14.2; no longer LED15.A2, R26.2
- net N$16: now also LED8.A3, R16.2; no longer LED15.A3, R33.2
- net N$19: now also LED8.A1, R18.2; no longer LED15.A1, R34.2
- net N$2: now also LED9.A, R17.2; no longer LED5.A, R3.2
- net N$3: now also LED10.A, R23.2; no longer LED6.A, R4.2
- net N$34: now also LED6.A, R12.2; no longer LED8.A, R27.2
- net N$35: now also LED7.A, R15.2; no longer LED9.A, R28.2
- net N$36: now also LED2.A, R2.2; no longer LED10.A, R29.2
- net N$37: now also LED4.A, R10.2; no longer LED11.A, R30.2
- net N$38: now also R1.2; no longer R31.2
- net N$39: now also R9.2; no longer R32.2
- net N$4: now also LED11.A, R24.2; no longer LED7.A, R7.2
- net N$5: now also LED5.C1, LED8.C1, Q3.6; no longer LED14.C1, LED15.C1, Q1.6
- net N$6: now also LED5.C3, LED8.C3, Q3.3; no longer LED14.C3, LED15.C3, Q1.3
- net N$7: now also LED5.C2, LED8.C2, Q6.6; no longer LED14.C2, LED15.C2, Q2.6
- net N$8: now also LED5.A2, R8.2; no longer LED14.A2, R10.2
- net N$9: now also LED5.A3, R11.2; no longer LED14.A3, R24.2
- net OSC-IN: now also C1.1, U1.5; no longer C15.1, U4.5
- net OSC-OUT: now also C2.1, U1.6; no longer C16.1, U4.6
- net OTG-HS-DM: now also U1.35; no longer U4.35
- net OTG-HS-DP: now also U1.36; no longer U4.36
- net OTG-HS-ID: now also U1.33; no longer U4.33
- net PA12: now also R17.1, U1.45; no longer R3.1, U4.45
- net PA15: now also R23.1, U1.50; no longer R4.1, U4.50
- net PA4: now also J3.1, U1.20; no longer J11.1, U4.20
- net PA5: now also J8.1, U1.21; no longer J12.1, U4.21
- net PB2: now also R24.1, U1.28; no longer R7.1, U4.28
- net PC4: now also J12.1, U1.24; no longer J21.1, U4.24
- net PC5: now also J15.1, U1.25; no longer J22.1, U4.25
- net RST: now also J21.1, R25.1, U1.7; no longer J20.1, R8.1, U4.7
- net SDIO-CK: now also U1.53, U5.5; no longer U3.5, U4.53
- net SDIO-CMD: now also U1.54, U5.3; no longer U3.3, U4.54
- net SDIO-D0: now also U1.39, U5.7; no longer U3.7, U4.39
- net SDIO-D1: now also U1.40, U5.8; no longer U3.8, U4.40
- net SDIO-D2: now also U1.51, U5.1; no longer U3.1, U4.51
- net SDIO-D3: now also U1.52, U5.2; no longer U3.2, U4.52
- net SPI1-MISO: now also R30.1, U1.56, U3.9; no longer R18.1, U4.56, U6.9
- net SPI1-MOSI: now also U1.57, U3.24; no longer U4.57, U6.24
- net SPI1-SCK: now also U1.55, U3.23; no longer U4.55, U6.23
- net SPI2-MISO: now also J18.2, R32.1, U1.10; no longer J15.2, R37.1, U4.10
- net SPI2-MOSI: now also J18.3, U1.11; no longer J15.3, U4.11
- net SPI2-SCK: now also J18.1, U1.34; no longer J15.1, U4.34
- net SPISS-MPU9250: now also U1.3, U3.22; no longer U4.3, U6.22
- net SPISS-MS5611: now also U1.2; no longer U4.2
- net SPISS-UNUSED: now also U1.4; no longer U4.4
- net SWCLK: now also J21.4, U1.49; no longer J20.4, U4.49
- net SWDIO: now also J21.3, U1.46; no longer J20.3, U4.46
- net TIM1-CH1: now also R4.2, U1.41; no longer R35.2, U4.41
- net TIM1-CH1-K: now also Q1.6, R4.1; no longer Q7.6, R35.1
- net TIM1-CH2: now also R5.2, U1.42; no longer R36.2, U4.42
- net TIM1-CH2-K: now also J6.1, Q1.3, R5.1; no longer J2.1, Q7.3, R36.1
- net TIM1-CH3: now also R6.2, U1.43; no longer R38.2, U4.43
- net TIM1-CH3-K: now also J10.1, Q2.6, R6.1; no longer J3.1, Q8.6, R38.1
- net TIM1-CH4: now also R7.2, U1.44; no longer R43.2, U4.44
- net TIM1-CH4-K: now also J13.1, Q2.3, R7.1; no longer J4.1, Q8.3, R43.1
- net TIM3-CH1-RSSI: now also R12.1, U1.22; no longer R27.1, U4.22
- net TIM3-CH2-STSR: now also Q6.2, U1.23; no longer Q2.2, U4.23
- net TIM3-CH3-STSG: now also Q3.5, U1.26; no longer Q1.5, U4.26
- net TIM3-CH4-STSB: now also Q3.2, U1.27; no longer Q1.2, U4.27
- net TIM4-CH1: now also U1.58; no longer U4.58
- net TIM4-CH1-K: now also J2.1; no longer J5.1
- net TIM4-CH2: now also U1.59; no longer U4.59
- net TIM4-CH2-K: now also J7.1; no longer J6.1
- net TIM4-CH3: now also U1.61; no longer U4.61
- net TIM4-CH3-K: now also J11.1; no longer J7.1
- net TIM4-CH4: now also U1.62; no longer U4.62
- net TIM4-CH4-K: now also J14.1; no longer J8.1
- net UART2-RX-XBEE: now also R10.1, U1.17; no longer R30.1, U4.17
- net UART2-TX-XBEE: now also R2.1, U1.16; no longer R29.1, U4.16
- net UART4-RX: now also J20.2, U1.15; no longer J19.2, U4.15
- net UART4-TX: now also J20.1, U1.14; no longer J19.1, U4.14
- net UART6-RX-GPS: now also J19.3, U1.38; no longer J18.3, U4.38
- net UART6-TX-GPS: now also J19.2, U1.37; no longer J18.2, U4.37
- net USD-CD: now also R34.1, U5.CD1, U5.CD2; no longer R2.1, U3.CD1, U3.CD2
- net VIN: now also J5.1, Q7.5, Q7.6, Q7.7, Q7.8; no longer J10.1, Q3.5, Q3.6, Q3.7, Q3.8

Commit message: Add test points.
Parts:
- added TP1, TP10, TP11, TP12, TP13, TP14, TP15, TP2, TP3, TP7, TP8, TP9: TEST-POINT-KEYSTONE-5019, OSURC_Passives:PAD.15X.08
- added TP4, TP5, TP6: TEST-POINT-PAD.03C, OSURC_Passives:PAD-.03C
Connections:
- new net BOOT0: TP1.1, U1.60
- net KILL: now also TP2.1
- net OTG-HS-DM: now also TP7.1
- net OTG-HS-DP: now also TP8.1
- net SDIO-CK: now also TP13.1
- net SDIO-CMD: now also TP14.1
- net SDIO-D0: now also TP9.1
- net SDIO-D1: now also TP10.1
- net SDIO-D2: now also TP11.1
- net SDIO-D3: now also TP12.1
- net SPI1-MISO: now also TP5.1
- net SPI1-MOSI: now also TP6.1
- net SPI1-SCK: now also TP4.1
- net TIM3-CH1-RSSI: now also TP3.1
Changed lines of the file:
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@@
 <element name="J12" library="aerial" package="MOLEX-2MM-MICROLATCH-2POS-RA" value="MOLEX-2POS" x="-273.05" y="-595.63"/>
 <element name="J15" library="aerial" package="MOLEX-2MM-MICROLATCH-2POS-RA" value="MOLEX-2POS" x="-280.67" y="-595.63"/>
+<element name="TP1" library="OSURC_Passives" package="PAD.15X.08" value="TEST-POINT-KEYSTONE-5019" x="-280.67" y="-601.98">
+<attribute name="DIGIKEY_PN" value="5019KCT-ND" x="-280.67" y="-601.98" size="1.778" layer="27" display="off"/>
+</element>
+<element name="TP2" library="OSURC_Passives" package="PAD.15X.08" value="TEST-POINT-KEYSTONE-5019" x="-280.67" y="-604.52">
+<attribute name="DIGIKEY_PN" value="5019KCT-ND" x="-280.67" y="-604.52" size="1.778" layer="27" display="off"/>
+</element>
+<element name="TP3" library="OSURC_Passives" package="PAD.15X.08" value="TEST-POINT-KEYSTONE-5019" x="-280.67" y="-607.06">
+<attribute name="DIGIKEY_PN" value="5019KCT-ND" x="-280.67" y="-607.06" size="1.778" layer="27" display="off"/>
+</element>
+<element name="TP7" library="OSURC_Passives" package="PAD.15X.08" value="TEST-POINT-KEYSTONE-5019" x="-280.67" y="-609.6">
+<attribute name="DIGIKEY_PN" value="5019KCT-ND" x="-280.67" y="-609.6" size="1.778" layer="27" display="off"/>
+</element>
+<element name="TP8" library="OSURC_Passives" package="PAD.15X.08" value="TEST-POINT-KEYSTONE-5019" x="-280.67" y="-612.14">
+<attribute name="DIGIKEY_PN" value="5019KCT-ND" x="-280.67" y="-612.14" size="1.778" layer="27" display="off"/>
+</element>
+<element name="TP9" library="OSURC_Passives" package="PAD.15X.08" value="TEST-POINT-KEYSTONE-5019" x="-280.67" y="-614.68">
+<attribute name="DIGIKEY_PN" value="5019KCT-ND" x="-280.67" y="-614.68" size="1.778" layer="27" display="off"/>
+</element>
+<element name="TP10" library="OSURC_Passives" package="PAD.15X.08" value="TEST-POINT-KEYSTONE-5019" x="-280.67" y="-617.22">
+<attribute name="DIGIKEY_PN" value="5019KCT-ND" x="-280.67" y="-617.22" size="1.778" layer="27" display="off"/>
+</element>
+<element name="TP11" library="OSURC_Passives" package="PAD.15X.08" value="TEST-POINT-KEYSTONE-5019" x="-280.67" y="-619.76">
+<attribute name="DIGIKEY_PN" value="5019KCT-ND" x="-280.67" y="-619.76" size="1.778" layer="27" display="off"/>
+</element>
+<element name="TP12" library="OSURC_Passives" package="PAD.15X.08" value="TEST-POINT-KEYSTONE-5019" x="-280.67" y="-622.3">
+<attribute name="DIGIKEY_PN" value="5019KCT-ND" x="-280.67" y="-622.3" size="1.778" layer="27" display="off"/>
+</element>
+<element name="TP13" library="OSURC_Passives" package="PAD.15X.08" value="TEST-POINT-KEYSTONE-5019" x="-280.67" y="-624.84">
+<attribute name="DIGIKEY_PN" value="5019KCT-ND" x="-280.67" y="-624.84" size="1.778" layer="27" display="off"/>
+</element>
+<element name="TP14" library="OSURC_Passives" package="PAD.15X.08" value="TEST-POINT-KEYSTONE-5019" x="-280.67" y="-627.38">
+<attribute name="DIGIKEY_PN" value="5019KCT-ND" x="-280.67" y="-627.38" size="1.778" layer="27" display="off"/>
+</element>
+<element name="TP4" library="OSURC_Passives" package="PAD-.03C" value="TEST-POINT-PAD.03C" x="-281.94" y="-629.92"/>
+<element name="TP5" library="OSURC_Passives" package="PAD-.03C" value="TEST-POINT-PAD.03C" x="-281.94" y="-632.46"/>
+<element name="TP6" library="OSURC_Passives" package="PAD-.03C" value="TEST-POINT-PAD.03C" x="-281.94" y="-635"/>
+<element name="TP15" library="OSURC_Passives" package="PAD.15X.08" value="TEST-POINT-KEYSTONE-5019" x="-280.67" y="-637.54">
+<attribute name="DIGIKEY_PN" value="5019KCT-ND" x="-280.67" y="-637.54" size="1.778" layer="27" display="off"/>
+</element>
 </elements>
 <signals>
@@
 <contactref element="Q2" pad="5"/>
 <contactref element="R3" pad="1"/>
+<contactref element="TP2" pad="1"/>
 <wire x1="22.8" y1="78.17" x2="-27.55" y2="-219.5" width="0" layer="19" extent="1-1"/>
-<wire x1="-223.27" y1="-560.7" x2="22.8" y2="78.17" width="0" layer="19" extent="1-1"/>
+<wire x1="-223.27" y1="-560.7" x2="-27.55" y2="-219.5" width="0" layer="19" extent="1-1"/>
 <wire x1="-224.73" y1="-560.7" x2="-223.27" y2="-560.7" width="0" layer="19" extent="1-1"/>
 <wire x1="-224.73" y1="-571.7" x2="-224.73" y2="-560.7" width="0" layer="19" extent="1-1"/>
 <wire x1="-223.27" y1="-571.7" x2="-224.73" y2="-571.7" width="0" layer="19" extent="1-1"/>
 <wire x1="-224.65" y1="-582.2" x2="-224.73" y2="-571.7" width="0" layer="19" extent="1-1"/>
+<wire x1="-280.67" y1="-604.52" x2="-224.65" y2="-582.2" width="0" layer="19" extent="1-1"/>
 </signal>
 <signal name="UART4-TX">
@@
 <contactref element="U2" pad="8"/>
 <contactref element="U3" pad="23"/>
-<wire x1="-186.2" y1="-460.525" x2="21.97" y2="23.99" width="0" layer="19" extent="1-1"/>
-<wire x1="-250.65" y1="-592.9" x2="-186.2" y2="-460.525" width="0" layer="19" extent="1-1"/>
+<contactref element="TP4" pad="1"/>
+<wire x1="-250.65" y1="-592.9" x2="-281.94" y2="-629.92" width="0" layer="19" extent="1-1"/>
+<wire x1="-186.2" y1="-460.525" x2="-250.65" y2="-592.9" width="0" layer="19" extent="1-1"/>
+<wire x1="21.97" y1="23.99" x2="-186.2" y2="-460.525" width="0" layer="19" extent="1-1"/>
 </signal>
 <signal name="SPI1-MOSI">
@@
 <contactref element="U2" pad="7"/>
 <contactref element="U3" pad="24"/>
-<wire x1="-186.2" y1="-461.775" x2="20.97" y2="23.99" width="0" layer="19" extent="1-1"/>
-<wire x1="-251.15" y1="-592.9" x2="-186.2" y2="-461.775" width="0" layer="19" extent="1-1"/>
+<contactref element="TP6" pad="1"/>
+<wire x1="-251.15" y1="-592.9" x2="-281.94" y2="-635" width="0" layer="19" extent="1-1"/>
+<wire x1="-186.2" y1="-461.775" x2="-251.15" y2="-592.9" width="0" layer="19" extent="1-1"/>
+<wire x1="20.97" y1="23.99" x2="-186.2" y2="-461.775" width="0" layer="19" extent="1-1"/>
 </signal>
 <signal name="SPI2-SCK">
@@
 <contactref element="U1" pad="36"/>
 <contactref element="JP1" pad="D+"/>
-<wire x1="-38.7" y1="-350.45" x2="27.17" y2="15.79" width="0" layer="19" extent="1-1"/>
+<contactref element="TP8" pad="1"/>
+<wire x1="-280.67" y1="-612.14" x2="-38.7" y2="-350.45" width="0" layer="19" extent="1-1"/>
+<wire x1="27.17" y1="15.79" x2="-38.7" y2="-350.45" width="0" layer="19" extent="1-1"/>
 </signal>
 <signal name="SPI1-MISO">
@@
 <contactref element="R30" pad="1"/>
 <contactref element="U3" pad="9"/>
+<contactref element="TP5" pad="1"/>
 <wire x1="-186.2" y1="-463.025" x2="-188.35" y2="-493.4" width="0" layer="19" extent="1-1"/>
 <wire x1="-250.15" y1="-596.9" x2="-188.35" y2="-493.4" width="0" layer="19" extent="1-1"/>
+<wire x1="-281.94" y1="-632.46" x2="-250.15" y2="-596.9" width="0" layer="19" extent="1-1"/>
 <wire x1="21.47" y1="23.99" x2="-186.2" y2="-463.025" width="0" layer="19" extent="1-1"/>
 </signal>
@@
 <contactref element="U1" pad="35"/>
 <contactref element="JP1" pad="D-"/>
-<wire x1="-39.35" y1="-350.45" x2="27.17" y2="15.29" width="0" layer="19" extent="1-1"/>
+<contactref element="TP7" pad="1"/>
+<wire x1="-280.67" y1="-609.6" x2="-39.35" y2="-350.45" width="0" layer="19" extent="1-1"/>
+<wire x1="27.17" y1="15.29" x2="-39.35" y2="-350.45" width="0" layer="19" extent="1-1"/>
 </signal>
 <signal name="SPI2-MISO">
@@
 <contactref element="U1" pad="51"/>
 <contactref element="U5" pad="1"/>
+<contactref element="TP11" pad="1"/>
+<wire x1="23.97" y1="23.99" x2="-280.67" y2="-619.76" width="0" layer="19" extent="1-1"/>
 <wire x1="41.36" y1="31.47" x2="23.97" y2="23.99" width="0" layer="19" extent="1-1"/>
 </signal>
@@
 <contactref element="U1" pad="52"/>
 <contactref element="U5" pad="2"/>
+<contactref element="TP12" pad="1"/>
+<wire x1="23.47" y1="23.99" x2="-280.67" y2="-622.3" width="0" layer="19" extent="1-1"/>
 <wire x1="42.46" y1="31.07" x2="23.47" y2="23.99" width="0" layer="19" extent="1-1"/>
 </signal>
@@
 <contactref element="U1" pad="53"/>
 <contactref element="U5" pad="5"/>
+<contactref element="TP13" pad="1"/>
+<wire x1="22.97" y1="23.99" x2="-280.67" y2="-624.84" width="0" layer="19" extent="1-1"/>
 <wire x1="45.76" y1="31.47" x2="22.97" y2="23.99" width="0" layer="19" extent="1-1"/>
 </signal>
@@
 <contactref element="U1" pad="54"/>
 <contactref element="U5" pad="3"/>
+<contactref element="TP14" pad="1"/>
+<wire x1="22.47" y1="23.99" x2="-280.67" y2="-627.38" width="0" layer="19" extent="1-1"/>
 <wire x1="43.56" y1="31.47" x2="22.47" y2="23.99" width="0" layer="19" extent="1-1"/>
 </signal>
@@
 <contactref element="U1" pad="39"/>
 <contactref element="U5" pad="7"/>
+<contactref element="TP9" pad="1"/>
+<wire x1="27.17" y1="17.29" x2="-280.67" y2="-614.68" width="0" layer="19" extent="1-1"/>
 <wire x1="47.96" y1="31.47" x2="27.17" y2="17.29" width="0" layer="19" extent="1-1"/>
 </signal>
@@
 <contactref element="U1" pad="40"/>
 <contactref element="U5" pad="8"/>
+<contactref element="TP10" pad="1"/>
+<wire x1="27.17" y1="17.79" x2="-280.67" y2="-617.22" width="0" layer="19" extent="1-1"/>
 <wire x1="49.06" y1="31.47" x2="27.17" y2="17.79" width="0" layer="19" extent="1-1"/>
 </signal>
@@
 <contactref element="R12" pad="1"/>
 <contactref element="XBEE" pad="6"/>
+<contactref element="TP3" pad="1"/>
 <wire x1="19.97" y1="12.09" x2="-30.65" y2="-219.5" width="0" layer="19" extent="1-1"/>
-<wire x1="3.8" y1="68.17" x2="-30.65" y2="-219.5" width="0" layer="19" extent="1-1"/>
+<wire x1="3.8" y1="68.17" x2="19.97" y2="12.09" width="0" layer="19" extent="1-1"/>
+<wire x1="-280.67" y1="-607.06" x2="-30.65" y2="-219.5" width="0" layer="19" extent="1-1"/>
 </signal>
 <signal name="N$5">
@@
 <wire x1="-244.25" y1="-595" x2="-249.65" y2="-596.9" width="0" layer="19" extent="1-1"/>
 </signal>
+<signal name="BOOT0">
+<contactref element="U1" pad="60"/>
+<contactref element="TP1" pad="1"/>
+<wire x1="19.47" y1="23.99" x2="-280.67" y2="-601.98" width="0" layer="19" extent="1-1"/>
+</signal>
 </signals>

Commit message: Update connectors with those from OSURC libs.
Dunno how these didn't get updated last time.
Parts:
- J10, J11, J12, J13, J14, J15, J2, J3, J5, J6, J7, J8: value MOLEX-2POS -> M02; device aerial:MOLEX-2MM-MICROLATCH-2POS-RA -> OSURC_Connectors:MOLEX-2MM-MICROLATCH-2POS-RA
- J16, J20, J4, J9: value MOLEX-3POS -> M03; device aerial:MOLEX-2MM-MICROLATCH-3POS-RA -> OSURC_Connectors:MOLEX-2MM-MICROLATCH-3POS-RA
- J18, J21: value MOLEX-4POS -> M04; device aerial:MOLEX-2MM-MICROLATCH-4POS-RA -> OSURC_Connectors:MOLEX-2MM-MICROLATCH-4POS-RA
- moved J1 370.7 mm to (-311.1, -633.7)
- moved J21 366.9 mm to (-416.6, -665.5)
- moved J9 361.4 mm to (-389.9, -633.7)
- moved J4 361.2 mm to (-381.0, -633.7)
- moved J17 355.9 mm to (-407.7, -633.7)
- moved J16 355.7 mm to (-398.8, -633.7)
- moved J14 353.6 mm to (-334.0, -633.7)
- moved J11 353.0 mm to (-326.4, -633.7)
- moved J7 352.5 mm to (-318.8, -633.7)
- moved J13 351.4 mm to (-303.5, -633.7)
- moved J10 350.8 mm to (-295.9, -633.7)
- moved J20 350.3 mm to (-416.6, -633.7)
- moved J6 350.3 mm to (-288.3, -633.7)
- moved J18 344.2 mm to (-416.6, -645.2)
- moved J19 247.3 mm to (-416.6, -655.3)
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Connections:
- net GND: now also J21.4; no longer J1.2, J21.2
- net SWCLK: now also J21.3; no longer J21.4
- net SWDIO: now also J21.2; no longer J21.3
- net TIM1-CH1-K: now also J2.1; no longer J1.1
- net TIM4-CH1-K: no longer J2.1
